Commit message: making it work

File: body.urdf (robot description, URDF)
Before this commit: robot robot, 3 links, 2 joints
Links:
- removed link BackLeg
- removed link FrontLeg
- added link BackArm, mass 1; collision box size=0.3 0.3 1; visual box size=0.3 0.3 1
- added link FrontArm, mass 1; collision box size=0.3 0.3 1; visual box size=0.3 0.3 1
- added link LeftArm, mass 1; collision box size=0.3 0.3 1; visual box size=0.3 0.3 1
- added link Leg, mass 1; collision box size=0.3 0.3 2; visual box size=0.3 0.3 2
- added link RightArm, mass 1; collision box size=0.3 0.3 1; visual box size=0.3 0.3 1
Joints:
- removed joint Torso_BackLeg
- removed joint Torso_FrontLeg
- added joint Torso_BackArm: type revolute, parent Torso, child BackArm, origin xyz=-0.5 0 3 rpy=0 0 0, axis 0 1 0, limit lower=-3.14159 upper=3.14159 effort=0.0 velocity=0.0
- added joint Torso_FrontArm: type revolute, parent Torso, child FrontArm, origin xyz=0.5 0 3 rpy=0 0 0, axis 0 1 0, limit lower=-3.14159 upper=3.14159 effort=0.0 velocity=0.0
- added joint Torso_LeftArm: type revolute, parent Torso, child LeftArm, origin xyz=0 0.5 3 rpy=0 0 0, axis 1 0 0, limit lower=-3.14159 upper=3.14159 effort=0.0 velocity=0.0
- added joint Torso_Leg: type revolute, parent Torso, child Leg, origin xyz=0 0 2.5 rpy=0 0 0, axis 0 1 0, limit lower=-3.14159 upper=3.14159 effort=0.0 velocity=0.0
- added joint Torso_RightArm: type revolute, parent Torso, child RightArm, origin xyz=0 -0.5 3 rpy=0 0 0, axis 1 0 0, limit lower=-3.14159 upper=3.14159 effort=0.0 velocity=0.0

Commit message: worms

File: body.urdf (robot description, URDF)
Before this commit: robot robot, 6 links, 5 joints
Links:
- removed link BackArm
- removed link FrontArm
- removed link LeftArm
- removed link Leg
- removed link RightArm
- removed link Torso
- added link 0, mass 1; collision box size=0.7828446916498412 0.8855118314549913 0.37748211231403217; visual box size=0.7828446916498412 0.8855118314549913 0.37748211231403217
- added link 1, mass 1; collision box size=0.7310267089303535 0.7882152018541339 0.22144500762364916; visual box size=0.7310267089303535 0.7882152018541339 0.22144500762364916
- added link 2, mass 1; collision box size=0.7669485124213186 0.766195148326613 0.07844524032296794; visual box size=0.7669485124213186 0.766195148326613 0.07844524032296794
- added link 3, mass 1; collision box size=0.4724735645661905 0.3760143203903804 0.23654833098921058; visual box size=0.4724735645661905 0.3760143203903804 0.23654833098921058
- added link 4, mass 1; collision box size=0.6524737309840533 0.8081653707573142 0.28832669196471805; visual box size=0.6524737309840533 0.8081653707573142 0.28832669196471805
Joints:
- removed joint Torso_BackArm
- removed joint Torso_FrontArm
- removed joint Torso_LeftArm
- removed joint Torso_Leg
- removed joint Torso_RightArm
- added joint 0_1: type revolute, parent 0, child 1, origin xyz=0 0.4427559157274957 0.11072250381182458 rpy=0 0 0, axis 1 0 0, limit lower=-3.14159 upper=3.14159 effort=0.0 velocity=0.0
- added joint 1_2: type revolute, parent 1, child 2, origin xyz=0 0.7882152018541339 -0.0714998836503406 rpy=0 0 0, axis 1 0 0, limit lower=-3.14159 upper=3.14159 effort=0.0 velocity=0.0
- added joint 2_3: type revolute, parent 2, child 3, origin xyz=0 0.766195148326613 0.07905154533312131 rpy=0 0 0, axis 1 0 0, limit lower=-3.14159 upper=3.14159 effort=0.0 velocity=0.0
- added joint 3_4: type revolute, parent 3, child 4, origin xyz=0 0.3760143203903804 0.025889180487753738 rpy=0 0 0, axis 1 0 0, limit lower=-3.14159 upper=3.14159 effort=0.0 velocity=0.0

Commit message: assignment 7

File: body.urdf (robot description, URDF)
Before this commit: robot robot, 5 links, 4 joints
Links:
- added link 10, mass 1; collision box size=0.7122663944550651 0.8767191117323297 0.7327257122493671; visual box size=0.7122663944550651 0.8767191117323297 0.7327257122493671
- added link 5, mass 1; collision box size=0.11135753165312388 0.10686242788024079 0.1697412837080099; visual box size=0.11135753165312388 0.10686242788024079 0.1697412837080099
- added link 6, mass 1; collision box size=0.08773858716176473 0.26955041443051675 0.5380362044694998; visual box size=0.08773858716176473 0.26955041443051675 0.5380362044694998
- added link 7, mass 1; collision box size=0.523210054589652 0.05390180663409538 0.06505370324381075; visual box size=0.523210054589652 0.05390180663409538 0.06505370324381075
- added link 8, mass 1; collision box size=0.96293937488655 0.801963275342113 0.0585349403823504; visual box size=0.96293937488655 0.801963275342113 0.0585349403823504
- added link 9, mass 1; collision box size=0.45953874601103684 0.8879719146668597 0.7197470145293705; visual box size=0.45953874601103684 0.8879719146668597 0.7197470145293705
- link 0: geometry collision box size=0.5060868132530039 0.42281782326665684 0.8442235609680201; visual box size=0.5060868132530039 0.42281782326665684 0.8442235609680201
- link 1: geometry collision box size=0.04704660608373223 0.5424710356899762 0.934802636479536; visual box size=0.04704660608373223 0.5424710356899762 0.934802636479536
- link 2: geometry collision box size=0.7014064301288392 0.751450437347119 0.9943286479224304; visual box size=0.7014064301288392 0.751450437347119 0.9943286479224304
- link 3: geometry collision box size=0.6492919287571762 0.35338094461142666 0.4177036520300148; visual box size=0.6492919287571762 0.35338094461142666 0.4177036520300148
- link 4: geometry collision box size=0.15778629912728404 0.5183753365567384 0.3405919957621396; visual box size=0.15778629912728404 0.5183753365567384 0.3405919957621396
Joints:
- added joint 4_5: type revolute, parent 4, child 5, origin xyz=0.2591876682783692 0.2591876682783692 0.0 rpy=0 0 0, axis 1 0 0, limit lower=-3.14159 upper=3.14159 effort=0.0 velocity=0.0
- added joint 5_6: type revolute, parent 5, child 6, origin xyz=0.0 0.10686242788024079 0.0 rpy=0 0 0, axis 1 0 0, limit lower=-3.14159 upper=3.14159 effort=0.0 velocity=0.0
- added joint 6_7: type revolute, parent 6, child 7, origin xyz=0.0 0.2690181022347499 0.2690181022347499 rpy=0 0 0, axis 1 0 0, limit lower=-3.14159 upper=3.14159 effort=0.0 velocity=0.0
- added joint 7_8: type revolute, parent 7, child 8, origin xyz=0.261605027294826 0.0 0.261605027294826 rpy=0 0 0, axis 0 1 0, limit lower=-3.14159 upper=3.14159 effort=0.0 velocity=0.0
- added joint 8_9: type revolute, parent 8, child 9, origin xyz=0.0292674701911752 0.0 0.0292674701911752 rpy=0 0 0, axis 1 0 0, limit lower=-3.14159 upper=3.14159 effort=0.0 velocity=0.0
- added joint 9_10: type revolute, parent 9, child 10, origin xyz=0.0 0.0 0.7197470145293705 rpy=0 0 0, axis 1 0 0, limit lower=-3.14159 upper=3.14159 effort=0.0 velocity=0.0
- joint 0_1: axis 1 0 0 -> 0 1 0; origin xyz=0 0.4427559157274957 0.11072250381182458 rpy=0 0 0 -> xyz=0.25304340662650193 0.0 0.0 rpy=0 0 0
- joint 1_2: origin xyz=0 0.7882152018541339 -0.0714998836503406 rpy=0 0 0 -> xyz=0.467401318239768 0.0 0.467401318239768 rpy=0 0 0
- joint 2_3: origin xyz=0 0.766195148326613 0.07905154533312131 rpy=0 0 0 -> xyz=0.0 0.3757252186735595 0.3757252186735595 rpy=0 0 0
- joint 3_4: axis 1 0 0 -> 0 1 0; origin xyz=0 0.3760143203903804 0.025889180487753738 rpy=0 0 0 -> xyz=0.3246459643785881 0.3246459643785881 0.0 rpy=0 0 0

Commit message: assignment 8

File: body.urdf (robot description, URDF)
Before this commit: robot robot, 11 links, 10 joints
Links:
- link 0: geometry collision box size=0.8051935655656967 0.7517869892607294 0.6329016948897019; visual box size=0.8051935655656967 0.7517869892607294 0.6329016948897019
- link 1: geometry collision box size=0.7859585674357169 0.25905265606175776 0.06185325369909766; visual box size=0.7859585674357169 0.25905265606175776 0.06185325369909766
- link 10: geometry collision box size=0.3199579316031288 0.8285180746470708 0.49074518663003897; visual box size=0.3199579316031288 0.8285180746470708 0.49074518663003897
- link 2: geometry collision box size=0.3817933555623072 0.8784454578650953 0.39075791704476515; visual box size=0.3817933555623072 0.8784454578650953 0.39075791704476515
- link 3: geometry collision box size=0.2593307144426866 0.7411837167794242 0.418151054974514; visual box size=0.2593307144426866 0.7411837167794242 0.418151054974514
- link 4: geometry collision box size=0.16960421235803824 0.8071469914312045 0.14876741839890317; visual box size=0.16960421235803824 0.8071469914312045 0.14876741839890317
- link 5: geometry collision box size=0.14224085421692467 0.9823372896865363 0.01531313724410809; visual box size=0.14224085421692467 0.9823372896865363 0.01531313724410809
- link 6: geometry collision box size=0.8824077654368019 0.2993051677469265 0.9714779889500835; visual box size=0.8824077654368019 0.2993051677469265 0.9714779889500835
- link 7: geometry collision box size=0.9509760010879991 0.7006419411069083 0.9765643123171954; visual box size=0.9509760010879991 0.7006419411069083 0.9765643123171954
- link 8: geometry collision box size=0.03157020837955126 0.4249067116227452 0.9457926558382951; visual box size=0.03157020837955126 0.4249067116227452 0.9457926558382951
- link 9: geometry collision box size=0.34185448722063816 0.8274003109567611 0.5961412585033709; visual box size=0.34185448722063816 0.8274003109567611 0.5961412585033709
Joints:
- joint 0_1: axis 0 1 0 -> 1 0 0; origin xyz=0.25304340662650193 0.0 0.0 rpy=0 0 0 -> xyz=0.0 0.0 0.31645084744485097 rpy=0 0 0
- joint 1_2: axis 1 0 0 -> 0 1 0; origin xyz=0.467401318239768 0.0 0.467401318239768 rpy=0 0 0 -> xyz=0.39297928371785845 0.0 0.39297928371785845 rpy=0 0 0
- joint 2_3: origin xyz=0.0 0.3757252186735595 0.3757252186735595 rpy=0 0 0 -> xyz=0.43922272893254766 0.43922272893254766 0.0 rpy=0 0 0
- joint 3_4: axis 0 1 0 -> 1 0 0; origin xyz=0.3246459643785881 0.3246459643785881 0.0 rpy=0 0 0 -> xyz=0.0 0.209075527487257 0.209075527487257 rpy=0 0 0
- joint 4_5: origin xyz=0.2591876682783692 0.2591876682783692 0.0 rpy=0 0 0 -> xyz=0.0 0.0 0.14876741839890317 rpy=0 0 0
- joint 5_6: origin xyz=0.0 0.10686242788024079 0.0 rpy=0 0 0 -> xyz=0.0 0.0 0.01531313724410809 rpy=0 0 0
- joint 6_7: origin xyz=0.0 0.2690181022347499 0.2690181022347499 rpy=0 0 0 -> xyz=0.0 0.14965258387346325 0.14965258387346325 rpy=0 0 0
- joint 7_8: axis 0 1 0 -> 1 0 0; origin xyz=0.261605027294826 0.0 0.261605027294826 rpy=0 0 0 -> xyz=0.0 0.4882821561585977 0.4882821561585977 rpy=0 0 0
- joint 8_9: origin xyz=0.0292674701911752 0.0 0.0292674701911752 rpy=0 0 0 -> xyz=0.0 0.0 0.9457926558382951 rpy=0 0 0
- joint 9_10: origin xyz=0.0 0.0 0.7197470145293705 rpy=0 0 0 -> xyz=0.0 0.0 0.5961412585033709 rpy=0 0 0
